File: power.kicad_sch (KiCad schematic)
At the start: 17 parts, among them J1 Conn_01x06_Pin, U13 LP5907MFX-3.0, U14 LP5907MFX-4.5, U3 LM66100DCK, U4 LP5907MFX-3.0, U5 TPS22918TDBVRQ1, U6 LP5907MFX-3.0

Commit message: LDO for RF
Connections:
- net 5V_F: now also U13.3 (EN)
- net GND: now also U13.2 (GND)
- net 3V0_RF: now reaches U13.5 (OUT)
Changed lines of the file:
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@@
+	)
+	(junction
+		(at 209.55 41.91)
+		(diameter 0)
+		(color 0 0 0 0)
 	)
 	(junction
@@
 	(wire
 		(pts
+			(xy 209.55 41.91) (xy 208.28 41.91)
+		)
+		(stroke
+			(width 0)
+			(type default)
+		)
+	)
+	(wire
+		(pts
 			(xy 46.99 69.85) (xy 44.45 69.85)
 		)
@@
 	(wire
 		(pts
+			(xy 209.55 44.45) (xy 213.36 44.45)
+		)
+		(stroke
+			(width 0)
+			(type default)
+		)
+	)
+	(wire
+		(pts
 			(xy 67.31 64.77) (xy 72.39 64.77)
 		)
@@
 	(wire
 		(pts
+			(xy 213.36 41.91) (xy 209.55 41.91)
+		)
+		(stroke
+			(width 0)
+			(type default)
+		)
+	)
+	(wire
+		(pts
 			(xy 107.95 83.82) (xy 107.95 80.01)
 		)
@@
 	(wire
 		(pts
+			(xy 209.55 44.45) (xy 209.55 41.91)
+		)
+		(stroke
+			(width 0)
+			(type default)
+		)
+	)
+	(wire
+		(pts
 			(xy 166.37 29.21) (xy 166.37 25.4)
 		)
@@
 		)
 	)
+	(wire
+		(pts
+			(xy 229.87 41.91) (xy 228.6 41.91)
+		)
+		(stroke
+			(width 0)
+			(type default)
+		)
+	)
 	(text "LC low-pass for PWR-2/4 ripple"
 		(exclude_from_sim no)
@@
 	(text "LDO for RF"
 		(exclude_from_sim no)
-		(at 221.234 55.372 0)
-		(effects
-			(font
-				(size 1.27 1.27)
+		(at 230.632 52.832 0)
+		(effects
+			(font
+				(size 1.27 1.27)
+			)
+		)
+	)
+	(global_label "3V0_RF"
+		(shape input)
+		(at 229.87 41.91 0)
+		(fields_autoplaced yes)
+		(effects
+			(font
+				(size 1.27 1.27)
+			)
+			(justify left)
+		)
+		(property "Intersheetrefs" "${INTERSHEET_REFS}"
+			(at 239.689 41.91 0)
+			(effects
+				(font
+					(size 1.27 1.27)
+				)
+				(justify left)
+				(hide yes)
 			)
 		)
@@
 	(global_label "5V_F"
 		(shape input)
-		(at 213.36 41.91 180)
+		(at 208.28 41.91 180)
 		(fields_autoplaced yes)
 		(effects
@@
 		)
 		(property "Intersheetrefs" "${INTERSHEET_REFS}"
-			(at 206.0205 41.91 0)
+			(at 200.9405 41.91 0)
 			(effects
 				(font
@@
 					(unit 1)
 				)
+			)
+		)
+	)
+	(symbol
+		(lib_id "power:GND")
+		(at 220.98 52.07 0)
+		(unit 1)
+		(exclude_from_sim no)
+		(in_bom yes)
+		(on_board yes)
+		(dnp no)
+		(fields_autoplaced yes)
+		(property "Reference" "#PWR038"
+			(at 220.98 58.42 0)
+			(effects
+				(font
+					(size 1.27 1.27)
+				)
+				(hide yes)
+			)
+		)
+		(property "Value" "GND"
+			(at 220.98 57.15 0)
+			(effects
+				(font
+					(size 1.27 1.27)
+				)
+			)
+		)
+		(property "Footprint" ""
+			(at 220.98 52.07 0)
+			(effects
+				(font
+					(size 1.27 1.27)
+				)
+				(hide yes)
+			)
+		)
+		(property "Datasheet" ""
+			(at 220.98 52.07 0)
+			(effects
+				(font
+					(size 1.27 1.27)
+				)
+				(hide yes)
+			)
+		)
+		(property "Description" "Power symbol creates a global label with name \"GND\" , ground"
+			(at 220.98 52.07 0)
+			(effects
+				(font
+					(size 1.27 1.27)
+				)
+				(hide yes)
+			)
+		)
+		(pin "1"
+		)
+		(instances
+			(project ""
+				(path "/45f99759-2553-47c9-8640-9aec1810c6cc/7b2d3bba-bbf7-4c7f-a096-b989c0e14168"
+					(reference "#PWR038")
+					(unit 1)
+				)

Commit message: MAR LDO
Parts:
- added C13, C14, C15, C4: 1uF, symbol Device:C
- added FB1: FerriteBead, symbol Device:FerriteBead
Connections:
- net 3V0_RF: now also FB1.2; no longer U13.5 (OUT)
- net 5V_F: now also U14.1 (IN), U14.3 (EN), C14.1, C4.1
- net GND: now also U14.2 (GND), C13.2, C14.2, C15.2, C4.2
- net 4V5_MAR: now reaches U14.5 (OUT)
- net 4V5_MAR: now also C15.1
- new net: C13.1, FB1.1, U13.5 (OUT)
Other:
- note added: "3V LDO: Main LNA/digital RF. Switched by master switch (SYS-2)."
- note removed: "LDO for RF"
