File: VIP_direct_sampling_board.kicad_pcb (KiCad board)
At the start: 2 copper layers, 11 parts

Commit message: Merging Branch to Main
Parts:
- added D1: GC6002-350A, Diode_SMD:D_SOD-523, F.Cu at (120.7, 88.4)
- added U11: DC4759J5020AHF-1, RF_Converter:Anaren_0805_2012Metric-6, F.Cu at (120.5, 85.4)
- added U15: LP5907MFX-3.0, Package_TO_SOT_SMD:SOT-23-5, F.Cu at (116.3, 77.0)
- added U16: LM66100DCK, Package_TO_SOT_SMD:SOT-363_SC-70-6, F.Cu at (121.0, 81.5)
- added U17: LP5907MFX-3.0, Package_TO_SOT_SMD:SOT-23-5, F.Cu at (116.3, 81.7)
- added U19: LP5907MFX-4.5, Package_TO_SOT_SMD:SOT-23-5, F.Cu at (116.3, 86.3)
- added U20: LP5907MFX-3.0, Package_TO_SOT_SMD:SOT-23-5, F.Cu at (116.3, 90.9)
- added X1: B3715, Filter:Filter_SAW_Epcos_DCC6C_3x3mm, F.Cu at (122.0, 77.2)
